File: KiCAD/Flight_Computer_V1.kicad_sch (KiCad schematic)
At the start: 27 parts, among them J1 Conn_01x04_Pin, J2 Conn_01x04_Pin, J3 DEBUG, Q1 PMOS, U1 ESP32-WROOM-32UE-N16, U2 W25Q16JVSSIQ, U3 BMI088, U4 MMC5983MA, U5 MS560702BA03-50, X1 FA-20H

Commit message: Changes
Parts:
- removed J3: DEBUG, Connector_PinHeader_2.54mm:PinHeader_1x04_P2.54mm_Vertical, symbol Connector:Conn_01x04_Pin
- added C10: 1uF, symbol Device:C
- added J3: Conn_01x06_Pin, symbol Connector:Conn_01x06_Pin
- added Q2, Q3: NMOS, symbol Simulation_SPICE:NMOS
- added R10, R4, R6, R8: 100k, symbol Device:R
- added R11, R7: 27k, symbol Device:R
- added R12: 10k, symbol Device:R
- added R5, R9: 1k, symbol Device:R
- added SW1: SW_SPST, symbol Switch:SW_SPST
- U1: value ESP32-WROOM-32UE-N16 -> ESP32-WROOM-32
Connections:
- net +3.3V: now also J3.6 (Pin_6), R12.2
- net GND: now also C10.2, J3.3 (Pin_3), Q2.3 (S), Q3.3 (S), R11.1, R4.2, R7.1, R8.2, SW1.1 (A)
- net MOS_A: now also Q2.1 (D), R6.2
- net MOS_B: now also Q3.1 (D), R10.2
- net RESET: now reaches U1.3 (EN)
- net RESET: now also C10.1, J3.2 (Pin_2), R12.1, SW1.2 (B)
- new net: Q3.2 (G), R9.2
- new net: Q2.2 (G), R5.2
- new net FIRE_A: R4.1, R5.1
- new net FIRE_B: R8.1, R9.1
- new net GPIO_0: J3.1 (Pin_1)
- new net RXD0: J3.5 (Pin_5)
- new net SENSE_A: R6.1, R7.2
- new net SENSE_B: R10.1, R11.2
- new net TXD0: J3.4 (Pin_4)
Other:
- note added: "BAROMETER"
- note added: "CONTINUITY"
- note added: "PROGRAMMER SOCKET"
- note added: "RESET BUTTON"
- note removed: "DEBUG CONNECTOR"
- note removed: "RESET/BOOT BUTTONS"
- note removed: "USBminiB"

Commit message: GPS, RF Receiver
Parts:
- added C11, C12, C14, C15: 47nF, symbol Device:C
- added C13: 0.22uF, symbol Device:C
- added R13: 56k, symbol Device:R
- added U2: MAX-M10M-00B, MOD18_MAX-M10M_UBL, symbol MAX-M10:MAX-M10M-00B
- added U?: CC1200RHBR, RHB0032E, symbol CC1200RHBR:CC1200RHBR
- renumbered U2 to U1, U1 to U3, U3 to U4, U4 to U5, U5 to U6
Connections:
- net +3.3V: now also C11.1, C12.1, C14.1, C15.1, U2.7 (V_IO), U2.8 (VCC), U?.1 (VDD_GUARD), U?.12 (DVDD), U?.13 (AVDD_IF), U?.15 (AVDD_RF), U?.5 (DVDD)
- net GND: now also C11.2, C12.2, C13.2, C14.2, C15.2, R13.1, U2.1 (GND), U2.10 (GND), U2.12 (GND), U?.32 (EXT_XOSC), U?.33 (GND)
- net MISO: now also U?.9 (SO_GPIO1)
- net MOSI: now also U?.7 (SI)
- net SCK: now also U?.8 (SCLK)
- new net: R13.2, U?.14 (RBIAS)
- new net: C13.1, U?.6 (DCPL)
- new net CS_RADIO: U?.11 (CS_N)
- new net RADIO_INT: U?.4 (GPIO2)
- new net RESET_N: U?.2 (RESET_N)
- new net RXD: U2.2 (TXD)
- new net TXD: U2.3 (RXD)
- no-connect marks 2 -> 14
Other:
- moved on the sheet: C1, C2, C6, C7, C8, C9, Q2, Q3, R10, R11, R4, R5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
