File: KiCAD/Flight_Computer_V1.kicad_sch (KiCad schematic)
At the start: 42 parts, among them IC1 ESP32-S2-MINI-2-N4R2, J1 Conn_01x04_Pin, J2 Conn_01x04_Pin, J3 Conn_01x06_Pin, J4 Conn_02x04_Odd_Even, Q1 PMOS, Q2 NMOS, Q3 NMOS, SW1 SW_SPST, U1 W25Q16JVSSIQ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

Commit message: update
Parts:
- removed SW1: SW_SPST, symbol Switch:SW_SPST
- added SW1: PTS636 SM50J SMTR LFS, GSPTS004102:SW_PTS636_CNK, symbol GSPTS004102:PTS636_SM50J_SMTR_LFS
- BT1: footprint (none) -> Connector_JST:JST_PH_B2B-PH-K_1x02_P2.00mm_Vertical
- C5, C6: footprint (none) -> Capacitor_SMD:C_0201_0603Metric
- CR1: footprint SOT23-5L_STM -> LD2980ABM33TR:SOT23-5L_STM
- IC1: footprint ESP32S2MINI2N4R2 -> ESP32-Mini:ESP32S2MINI2N4R2
- J1, J2: footprint (none) -> 1725672:CONN_1725672_PXC
- J3: footprint (none) -> Connector_PinSocket_2.54mm:PinSocket_1x06_P2.54mm_Vertical
- J4: footprint (none) -> Connector_PinSocket_2.54mm:PinSocket_2x04_P2.54mm_Vertical
- Q1: footprint (none) -> Reverse Polarity PMOS:DMP3099L-7_DIO
- Q2, Q3: footprint SOT-23_MCC -> SI2302-TP:SOT-23_MCC
- R10, R9: footprint (none) -> Resistor_SMD:R_0201_0603Metric
- U1: footprint W25Q16JVSSIQ_WIN -> W25Q16JVSSIQ:W25Q16JVSSIQ_WIN
- U2: footprint MOD18_MAX-M10M_UBL -> MAX-M10:MOD18_MAX-M10M_UBL
- U4: footprint QFN_BMI085_BOS -> BMI088:QFN_BMI085_BOS
- U5: footprint MMC5983MA_MEM -> MMC5983MA:MMC5983MA_MEM
- U6: footprint SON8_MS5611_TEC -> MS560702BA03:SON8_MS5611_TEC
- X1: footprint XTAL4P_FA-20H_EPS -> FA-20H:XTAL4P_FA-20H_EPS
Connections:
- net GND: now also J3.5 (Pin_5), Q1.1 (G), SW1.1; no longer J3.4 (Pin_4), Q1.2 (G)
- net LiPO: now also Q1.2 (S); no longer Q1.1 (D)
- net RESET: now also J3.4 (Pin_4), SW1.2; no longer J3.5 (Pin_5)
- net RXD0: now also J3.3 (Pin_3); no longer J3.2 (Pin_2)
- net TXD0: now also J3.2 (Pin_2); no longer J3.3 (Pin_3)
Other:
- moved on the sheet: BT1, C4, Q1, R4

Commit message: V1 for review
Parts:
- added H1, H2, H3, H4: MountingHole_Pad, MountingHole:MountingHole_2.5mm_Pad, symbol Mechanical:MountingHole_Pad
- added TP1, TP2: TestPoint, TestPoint:TestPoint_Pad_D2.5mm, symbol Connector:TestPoint
- added TP3, TP4, TP5, TP6, TP7, TP8, TP9: TestPoint, TestPoint:TestPoint_Loop_D1.80mm_Drill1.0mm_Beaded, symbol Connector:TestPoint
Connections:
- net +3.3V: now also TP1.1
- net +BATT: now also TP2.1
- net ACCEL_INT: now also IC1.24 (IO20)
- net CS_ACCEL: now also IC1.23 (IO19)
- net CS_BARO: now also IC1.28 (IO33)
- net CS_FLASH: now also IC1.38 (IO42)
- net CS_GPS: now also IC1.41 (IO45)
- net CS_GYRO: now also IC1.26 (IO26)
- net CS_MAG: now also IC1.30 (GND_3)
- net FIRE_A: now also IC1.19 (IO15), TP6.1
- net FIRE_B: now also IC1.20 (IO16), TP7.1
- net GND: now also H1.1, H2.1, H3.1, H4.1
- net GYRO_INT: now also IC1.25 (IO21)
- net LiPO: no longer J2.2 (Pin_2)
- net MAG_INT: now also IC1.29 (IO34)
- net MISO: now also TP3.1
- net MOSI: now also TP4.1
- net MOS_LIPO: now also J2.2 (Pin_2)
- net PROGRAM_LED: now also IC1.34 (IO38)
- net RXD0: now also IC1.39 (TXD0), J3.2 (Pin_2); no longer IC1.40 (RXD0), J3.3 (Pin_3)
- net RXD1: now also IC1.21 (IO17), TP8.1
- net SCK: now also TP5.1
- net SENSE_A: now also IC1.17 (IO13)
- net SENSE_B: now also IC1.18 (IO14)
- net TXD0: now also IC1.40 (RXD0), J3.3 (Pin_3); no longer IC1.39 (TXD0), J3.2 (Pin_2)
- net TXD1: now also IC1.22 (IO18), TP9.1
Other:
- note added: "TEST POINTS"
- moved on the sheet: BT1, Q1

Commit message: Changes
Parts:
- added C11: 0.1uF, Capacitor_SMD:C_0201_0603Metric, symbol Device:C
- added GPS_ANT1: Conn_01x01, symbol Connector_Generic:Conn_01x01
- added TP10, TP11, TP12, TP14, TP15: TestPoint, TestPoint:TestPoint_Loop_D1.80mm_Drill1.0mm_Beaded, symbol Connector:TestPoint
Connections:
- net MOS_LIPO is gone; now on net RAW_BATT: J1.1 (Pin_1), J2.2 (Pin_2), Q1.3 (D)
- net +3.3V: now also C11.1
- net +BATT: now also Q1.2 (S)
- net CS_ACCEL: now also TP10.1
- net CS_BARO: now also TP12.1
- net CS_FLASH: now also TP14.1
- net CS_GYRO: now also TP11.1
- net GND: now also IC1.42 (GND_4), IC1.43 (GND_5), C11.2
- net MISO: now also J4.7 (Pin_7); no longer J4.5 (Pin_5)
- net MOSI: now also J4.6 (Pin_6); no longer J4.3 (Pin_3)
- net SCK: now also J4.5 (Pin_5); no longer J4.4 (Pin_4)
- net CS_GPS: no longer names the net of J4.8 (Pin_8)
- net CS_GPS: no longer IC1.41 (IO45)
- net GD0: no longer names the net of U2.11 (RF_IN)
- net GD0: now also GPS_ANT1.1 (Pin_1); no longer J4.7 (Pin_7)
- net GYRO_INT: no longer names the net of U4.12 (INT3)
- net GYRO_INT: no longer IC1.25 (IO21)
- net LiPO renamed RAW_BATT
- net RAW_BATT: no longer Q1.2 (S)
- new net CS_RF: IC1.41 (IO45), J4.4 (Pin_4), TP15.1
- new net GD00: J4.3 (Pin_3)
- no-connect marks 13 -> 30
Other:
- note added: "GPS ANTENNA"
- moved on the sheet: BT1, Q1, TP1, TP2, TP3, TP4, TP5, TP6, TP7, TP8, TP9, U1
