File: KiCAD/Flight_Computer_V1.kicad_pcb (KiCad board)
At the start: 2 copper layers, 36.8 x 50.8 mm, 42 parts, among them IC1 ESP32-S2-MINI-2-N4R2, J1 Conn_01x04_Pin, J2 Conn_01x04_Pin, J3 Conn_01x06_Pin, J4 Conn_02x04_Odd_Even, Q1 PMOS, Q2 NMOS, Q3 NMOS, SW1 PTS636 SM50J SMTR LFS, U1 W25Q16JVSSIQ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

Commit message: V1 for review
Parts:
- removed C2, C3: 22pF, Capacitor_SMD:C_0201_0603Metric
- removed X1: FA-20H, FA-20H:XTAL4P_FA-20H_EPS
- added H1: MountingHole_Pad, MountingHole:MountingHole_2.5mm_Pad, F.Cu at (18.4, 75.4)
- added H2: MountingHole_Pad, MountingHole:MountingHole_2.5mm_Pad, F.Cu at (18.5, 18.5)
- added H3: MountingHole_Pad, MountingHole:MountingHole_2.5mm_Pad, F.Cu at (48.8, 18.5)
- added H4: MountingHole_Pad, MountingHole:MountingHole_2.5mm_Pad, F.Cu at (48.8, 75.4)
- added TP1: TestPoint, TestPoint:TestPoint_Pad_D2.5mm, F.Cu at (48.3, 26.0)
- added TP2: TestPoint, TestPoint:TestPoint_Pad_D2.5mm, F.Cu at (44.0, 22.6)
- added TP3: TestPoint, TestPoint:TestPoint_Loop_D1.80mm_Drill1.0mm_Beaded, F.Cu at (35.2, 75.5)
- added TP4: TestPoint, TestPoint:TestPoint_Loop_D1.80mm_Drill1.0mm_Beaded, F.Cu at (31.4, 75.5)
- added TP5: TestPoint, TestPoint:TestPoint_Loop_D1.80mm_Drill1.0mm_Beaded, F.Cu at (39.0, 75.5)
- added TP6: TestPoint, TestPoint:TestPoint_Loop_D1.80mm_Drill1.0mm_Beaded, F.Cu at (33.4, 21.0)
- added TP7: TestPoint, TestPoint:TestPoint_Loop_D1.80mm_Drill1.0mm_Beaded, F.Cu at (38.1, 21.0)
- added TP8: TestPoint, TestPoint:TestPoint_Loop_D1.80mm_Drill1.0mm_Beaded, F.Cu at (27.6, 75.5)
- added TP9: TestPoint, TestPoint:TestPoint_Loop_D1.80mm_Drill1.0mm_Beaded, F.Cu at (23.8, 75.5)
- moved R10 106.5 mm to (19.3, 41.1), turned to 180 degrees
- moved R9 106.1 mm to (19.3, 42.0), turned to 180 degrees
- moved R11 104.6 mm to (22.6, 36.5), turned to 90 degrees
- moved BT1 104.2 mm to (26.1, 18.7)
- moved R12 104.0 mm to (23.6, 36.5), turned to -90 degrees
- moved C10 98.2 mm to (22.2, 48.9), turned to -90 degrees
- moved R6 96.8 mm to (27.5, 41.1), turned to 180 degrees
- moved U5 96.3 mm to (31.6, 60.4)
- moved R5 96.2 mm to (27.5, 42.1), turned to 180 degrees
- moved R7 95.1 mm to (30.9, 36.6), turned to 90 degrees
- moved R8 94.7 mm to (31.9, 36.6), turned to -90 degrees
- moved C7 90.2 mm to (29.9, 46.1), turned to 90 degrees
- moved C8 90.0 mm to (29.4, 59.7), turned to 90 degrees
- moved D3 88.5 mm to (41.5, 54.8), turned to 180 degrees
- moved D2 87.6 mm to (42.0, 32.5), turned to 90 degrees
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Connections:
- IC1 pad 17: unconnected-(IC1-IO13-Pad17) -> SENSE_A
- IC1 pad 18: unconnected-(IC1-IO14-Pad18) -> SENSE_B
- IC1 pad 19: unconnected-(IC1-IO15-Pad19) -> FIRE_A
- IC1 pad 20: unconnected-(IC1-IO16-Pad20) -> FIRE_B
- IC1 pad 21: unconnected-(IC1-IO17-Pad21) -> RXD1
- IC1 pad 22: unconnected-(IC1-IO18-Pad22) -> TXD1
- IC1 pad 23: unconnected-(IC1-IO19-Pad23) -> CS_ACCEL
- IC1 pad 24: unconnected-(IC1-IO20-Pad24) -> ACCEL_INT
- IC1 pad 25: unconnected-(IC1-IO21-Pad25) -> GYRO_INT
- IC1 pad 26: unconnected-(IC1-IO26-Pad26) -> CS_GYRO
- IC1 pad 28: unconnected-(IC1-IO33-Pad28) -> CS_BARO
- IC1 pad 29: unconnected-(IC1-IO34-Pad29) -> MAG_INT
- IC1 pad 30: unconnected-(IC1-GND_3-Pad30) -> CS_MAG
- IC1 pad 34: unconnected-(IC1-IO38-Pad34) -> PROGRAM_LED
- IC1 pad 38: unconnected-(IC1-IO42-Pad38) -> CS_FLASH
- IC1 pad 39: TXD0 -> RXD0
- IC1 pad 40: RXD0 -> TXD0
- IC1 pad 41: unconnected-(IC1-IO45-Pad41) -> CS_GPS
- J2 pad 2: LiPO -> MOS_LIPO
- J3 pad 2: TXD0 -> RXD0
- J3 pad 3: RXD0 -> TXD0
Routing:
- net MISO: track 0.00 -> 102.7 mm, vias 0 -> 2
- net MOSI: track 0.00 -> 87.3 mm, vias 0 -> 4
- net SCK: track 0.00 -> 85.9 mm, vias 0 -> 3
- net RXD1: track 0.00 -> 47.2 mm, vias 0 -> 3
- net GPIO_0: track 0.00 -> 46.6 mm
- net TXD1: track 0.00 -> 45.2 mm, vias 0 -> 3
- net FIRE_B: track 0.00 -> 41.1 mm, vias 0 -> 1
- net +BATT: track 0.00 -> 39.3 mm
- net GND: track 0.00 -> 32.1 mm, vias 0 -> 27
- net FIRE_A: track 0.00 -> 31.8 mm, vias 0 -> 1
- net CS_GPS: track 0.00 -> 30.4 mm, vias 0 -> 2
- net GD0: track 0.00 -> 29.4 mm
- net +3.3V: track 0.00 -> 24.6 mm, vias 0 -> 10
- net RESET: track 0.00 -> 21.8 mm
- net MOS_LIPO: track 0.00 -> 21.0 mm
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- added copper zone on In1.Cu, net +3.3V
- added copper zone on F.Cu, net GND
- added copper zone on In2.Cu, net GND
Other:
- board size 36.8 x 50.8 mm -> 36.8 x 63.5 mm
- copper layers 2 -> 4
- board text added: "+"
- board text added: "+3.3V"
- board text added: "+5V"
- board text added: "-"
- board text added: "APOGEE"
- board text added: "BATT"
- board text added: "FIRE_A"
- board text added: "FIRE_B"
- board text added: "GND"
- board text added: "GPIO0"
- board text added: "IN"
- board text added: "MAIN"
- board text added: "MISO"
- board text added: "MOSI"
- board text added: "OUT"
- board text added: "RST"
- board text added: "RXD"
- board text added: "RXD1"
- board text added: "SCK"
- board text added: "SWITCH"
- board text added: "TXD"
- board text added: "TXD1"

Commit message: Changes
Parts:
- added C11: 0.1uF, Capacitor_SMD:C_0201_0603Metric, F.Cu at (56.9, 56.1)
- added G***: LOGO, graphics:theone, F.Cu at (24.3, 30.2)
- added GPS_ANT: Pin_D1.0mm_L10.0mm, Connector_Pin:Pin_D1.0mm_L10.0mm, F.Cu at (24.4, 52.5)
- added TP10: TestPoint, TestPoint:TestPoint_Loop_D1.80mm_Drill1.0mm_Beaded, F.Cu at (29.9, 39.7)
- added TP11: TestPoint, TestPoint:TestPoint_Loop_D1.80mm_Drill1.0mm_Beaded, F.Cu at (24.8, 39.7)
- added TP12: TestPoint, TestPoint:TestPoint_Loop_D1.80mm_Drill1.0mm_Beaded, F.Cu at (19.7, 39.7)
- added TP14: TestPoint, TestPoint:TestPoint_Loop_D1.80mm_Drill1.0mm_Beaded, F.Cu at (59.8, 75.6)
- added TP15: TestPoint, TestPoint:TestPoint_Loop_D1.80mm_Drill1.0mm_Beaded, F.Cu at (37.1, 75.7)
- moved TP1 18.1 mm to (66.4, 25.8)
- moved H3 17.9 mm to (66.7, 18.5)
- moved H4 17.9 mm to (66.7, 75.4)
- moved SW1 17.1 mm to (66.5, 57.8)
- moved BT1 17.1 mm to (43.2, 18.8)
- moved C1 17.1 mm to (58.0, 26.5)
- moved C4 17.1 mm to (63.9, 54.9)
- moved C5 17.1 mm to (64.4, 35.2)
- moved C7 17.1 mm to (47.0, 46.2)
- moved C8 17.1 mm to (46.5, 59.8)
- moved C9 17.1 mm to (51.7, 60.3)
- moved D1 17.1 mm to (60.3, 32.6)
- moved D2 17.1 mm to (59.1, 32.6)
- moved D3 17.1 mm to (58.6, 54.9)
- moved IC1 17.1 mm to (59.8, 44.3)
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Connections:
- BT1 pad 1: LiPO -> RAW_BATT
- IC1 pad 25: GYRO_INT -> unconnected-(IC1-IO21-Pad25)
- IC1 pad 41: CS_GPS -> CS_RF
- IC1 pad 42: unconnected-(IC1-GND_4-Pad42) -> GND
- IC1 pad 43: unconnected-(IC1-GND_5-Pad43) -> GND
- J1 pad 1: MOS_LIPO -> RAW_BATT
- J2 pad 2: MOS_LIPO -> RAW_BATT
- J4 pad 3: MOSI -> GD00
- J4 pad 4: SCK -> CS_RF
- J4 pad 5: MISO -> SCK
- J4 pad 6: unconnected-(J4-Pin_6-Pad6) -> MOSI
- J4 pad 7: GD0 -> MISO
- J4 pad 8: CS_GPS -> unconnected-(J4-Pin_8-Pad8)
- Q1 pad 2: LiPO -> +BATT
- Q1 pad 3: MOS_LIPO -> RAW_BATT
- U2 pad 11: GD0 -> Net-(GPS_ANT1-Pin_1)
- U4 pad 12: GYRO_INT -> unconnected-(U4-INT3-Pad12)
Routing:
- net CS_RF: track 0.00 -> 65.7 mm, vias 0 -> 2
- net RAW_BATT: track 0.00 -> 37.3 mm
- net CS_GPS: track 30.4 -> 0.00 mm, vias 2 -> 0
- net GD0: track 29.4 -> 0.00 mm
- net CS_GYRO: track 7.27 -> 35.1 mm, vias 0 -> 1
- net CS_FLASH: track 15.8 -> 39.1 mm, vias 0 -> 1
- net CS_BARO: track 18.8 -> 41.8 mm
- net MOS_LIPO: track 21.0 -> 0.00 mm
- net CS_ACCEL: track 10.9 -> 27.5 mm, vias 0 -> 1
- net MOSI: track 87.3 -> 102.5 mm
- net LiPO: track 12.9 -> 0.00 mm
- net Net-(U2-RF_IN): track 0.00 -> 12.3 mm
- net GYRO_INT: track 11.1 -> 0.00 mm
- net MISO: track 102.7 -> 97.0 mm
- net SCK: track 85.9 -> 81.7 mm
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- added copper zone on In2.Cu, net +3.3V
- added copper zone on In1.Cu, net GND
- removed copper zone on In1.Cu, net +3.3V
- removed copper zone on In2.Cu, net GND
Other:
- board size 36.8 x 63.5 mm -> 54.6 x 63.5 mm
- board text added: "CS_ACC"
- board text added: "CS_BAR"
- board text added: "CS_FLASH"
- board text added: "CS_GYR"
- board text added: "CS_RF"
- board text added: "FLIGHT COMPUTER DEV"
- board text added: "GPS ANTENNA"
- board text added: "V1 - TEST"
