File: V2/Flight-Computer_V2.kicad_pcb (KiCad board)
At the start: 4 copper layers, 0 parts

Commit message: v2 cahnges
Parts:
- added BT1: LiPO, Connector_JST:JST_PH_B2B-PH-K_1x02_P2.00mm_Vertical, B.Cu at (42.3, 27.5)
- added C1: 22uF, Capacitor_SMD:C_0603_1608Metric, F.Cu at (117.0, 30.9)
- added C10: 0.1uF, Capacitor_SMD:C_0402_1005Metric, F.Cu at (118.9, 75.5)
- added C11: 0.1uF, Capacitor_SMD:C_0402_1005Metric, F.Cu at (118.9, 77.5)
- added C4: 1uF, Capacitor_SMD:C_0402_1005Metric, F.Cu at (118.9, 67.6)
- added C5: 10uF, Capacitor_SMD:C_0603_1608Metric, F.Cu at (117.0, 33.4)
- added C6: 0.1uF, Capacitor_SMD:C_0603_1608Metric, F.Cu at (117.0, 35.9)
- added C7: 0.1uF, Capacitor_SMD:C_0402_1005Metric, F.Cu at (118.9, 69.6)
- added C8: 1uF, Capacitor_SMD:C_0402_1005Metric, F.Cu at (118.9, 71.6)
- added C9: 10uF, Capacitor_SMD:C_0402_1005Metric, F.Cu at (118.9, 73.5)
- added CR1: LD2980ABM33TR, LD2980ABM33TR:SOT23-5L_STM, F.Cu at (115.6, 57.9)
- added D1: RED, LED_SMD:LED_0201_0603Metric, F.Cu at (119.0, 61.1)
- added D2: GREEN, LED_SMD:LED_0201_0603Metric, F.Cu at (119.0, 62.8)
- added D3: BLUE, LED_SMD:LED_0201_0603Metric, F.Cu at (119.0, 64.6)
- added H1: MountingHole_Pad, MountingHole:MountingHole_2.5mm_Pad, F.Cu at (29.2, 29.2)
- added H2: MountingHole_Pad, MountingHole:MountingHole_2.5mm_Pad, F.Cu at (76.5, 60.7)
- added H3: MountingHole_Pad, MountingHole:MountingHole_2.5mm_Pad, F.Cu at (76.5, 67.3)
- added H4: MountingHole_Pad, MountingHole:MountingHole_2.5mm_Pad, F.Cu at (76.5, 73.8)
- added J1: Conn_01x04_Pin, 1725672:CONN_1725672_PXC, B.Cu at (48.0, 33.2)
- added J2: Conn_01x04_Pin, 1725672:CONN_1725672_PXC, B.Cu at (34.5, 33.3)
- added J3: Conn_01x06_Pin, Connector_PinSocket_2.54mm:PinSocket_1x06_P2.54mm_Vertical, F.Cu at (96.1, 32.0)
- added J4: Conn_02x04_Odd_Even, Connector_PinSocket_2.54mm:PinSocket_2x04_P2.54mm_Vertical, F.Cu at (112.7, 32.0)
- added J5: 2337019-1, ul_2337019-1:CONN_2337019-1_TEC, F.Cu at (83.9, 73.8)
- added Q1: DMP3099L-7, Reverse Polarity PMOS:DMP3099L-7_DIO, F.Cu at (41.3, 37.5)
- added Q2: NMOS, SI2302-TP:SOT-23_MCC-M, F.Cu at (114.9, 69.6)
- added Q3: NMOS, SI2302-TP:SOT-23_MCC-M, F.Cu at (114.9, 75.5)
- added R1: 110, Resistor_SMD:R_0402_1005Metric, F.Cu at (99.8, 41.0)
- added R10: 1k, Resistor_SMD:R_0402_1005Metric, F.Cu at (102.8, 49.0)
- added R11: 100k, Resistor_SMD:R_0402_1005Metric, F.Cu at (105.7, 41.0)
- added R12: 27k, Resistor_SMD:R_0402_1005Metric, F.Cu at (105.7, 43.0)
- added R13: 10k, Resistor_SMD:R_0402_1005Metric, F.Cu at (105.7, 45.0)
- added R14: 10k, Resistor_SMD:R_0402_1005Metric, F.Cu at (105.7, 47.0)
- added R2: 50, Resistor_SMD:R_0402_1005Metric, F.Cu at (99.8, 43.0)
- added R3: 50, Resistor_SMD:R_0402_1005Metric, F.Cu at (99.8, 45.0)
- added R4: 10k, Resistor_SMD:R_0402_1005Metric, F.Cu at (99.8, 47.0)
- added R5: 100k, Resistor_SMD:R_0402_1005Metric, F.Cu at (99.8, 49.0)
- added R6: 1k, Resistor_SMD:R_0402_1005Metric, F.Cu at (102.8, 41.0)
- added R7: 100k, Resistor_SMD:R_0402_1005Metric, F.Cu at (102.8, 43.0)
- added R8: 27k, Resistor_SMD:R_0402_1005Metric, F.Cu at (102.8, 45.0)
- added R9: 100k, Resistor_SMD:R_0402_1005Metric, F.Cu at (102.8, 47.0)
- added SW1: PTS636 SM50J SMTR LFS, GSPTS004102:SW_PTS636_CNK, F.Cu at (103.3, 32.2)
- added SW2: PTS636 SM50J SMTR LFS, GSPTS004102:SW_PTS636_CNK, F.Cu at (103.3, 37.4)
- added TP1: TestPoint, TestPoint:TestPoint_Pad_D2.5mm, F.Cu at (90.0, 67.1)
- added TP10: TestPoint, TestPoint:TestPoint_Loop_D1.80mm_Drill1.0mm_Beaded, F.Cu at (91.4, 57.9)
- added TP11: TestPoint, TestPoint:TestPoint_Loop_D1.80mm_Drill1.0mm_Beaded, F.Cu at (91.4, 62.5)
- added TP12: TestPoint, TestPoint:TestPoint_Loop_D1.80mm_Drill1.0mm_Beaded, F.Cu at (96.1, 53.2)
- added TP14: TestPoint, TestPoint:TestPoint_Loop_D1.80mm_Drill1.0mm_Beaded, F.Cu at (96.1, 57.9)
- added TP15: TestPoint, TestPoint:TestPoint_Loop_D1.80mm_Drill1.0mm_Beaded, F.Cu at (96.1, 62.5)
- added TP2: TestPoint, TestPoint:TestPoint_Pad_D2.5mm, F.Cu at (90.0, 71.7)
- added TP3: TestPoint, TestPoint:TestPoint_Loop_D1.80mm_Drill1.0mm_Beaded, F.Cu at (82.1, 53.2)
- added TP4: TestPoint, TestPoint:TestPoint_Loop_D1.80mm_Drill1.0mm_Beaded, F.Cu at (82.1, 57.9)
- added TP5: TestPoint, TestPoint:TestPoint_Loop_D1.80mm_Drill1.0mm_Beaded, F.Cu at (82.1, 62.5)
- added TP6: TestPoint, TestPoint:TestPoint_Loop_D1.80mm_Drill1.0mm_Beaded, F.Cu at (86.8, 53.2)
- added TP7: TestPoint, TestPoint:TestPoint_Loop_D1.80mm_Drill1.0mm_Beaded, F.Cu at (86.8, 57.9)
- added TP8: TestPoint, TestPoint:TestPoint_Loop_D1.80mm_Drill1.0mm_Beaded, F.Cu at (86.8, 62.5)
- added TP9: TestPoint, TestPoint:TestPoint_Loop_D1.80mm_Drill1.0mm_Beaded, F.Cu at (91.4, 53.2)
- added U1: W25Q16JVSSIQ, W25Q16JVSSIQ:W25Q16JVSSIQ_WIN, F.Cu at (113.1, 45.4)
- added U2: MAX-M10M-00B, MAX-M10:MOD18_MAX-M10M_UBL, F.Cu at (105.4, 72.5)
- added U3: ESP32-WROOM-32UE, RF_Module:ESP32-WROOM-32UE, F.Cu at (41.5, 104.2)
- added U4: BMI088, BMI088:QFN_BMI085_BOS, F.Cu at (116.0, 53.2)
- added U5: MMC5983MA, MMC5983MA:MMC5983MA_MEM, F.Cu at (94.8, 74.2)
- added U6: MS560702BA03-50, MS560702BA03:SON8_MS5611_TEC, F.Cu at (95.3, 68.3)
Routing:
- net RAW_BATT: track 0.00 -> 0.85 mm
- added copper zone on F.Cu, net +BATT
Other:
- board outline added: 31.8 x 88.9 mm

Commit message: V2 Changes
Parts:
- D1, D2, D3: footprint LED_SMD:LED_0201_0603Metric -> LED_SMD:LED_0402_1005Metric
- J3, J4, J5, TP1, TP2: moved to B.Cu
- Q1: footprint Reverse Polarity PMOS:DMP3099L-7_DIO -> DMP3099L-7:DMP3099L-7_DIO
- TP10, TP11, TP12, TP14, TP15, TP3, TP4, TP5, TP6, TP7, TP8, TP9: footprint TestPoint:TestPoint_Loop_D1.80mm_Drill1.0mm_Beaded -> TestPoint:TestPoint_Loop_D2.60mm_Drill1.6mm_Beaded; moved to B.Cu
- moved C5 103.7 mm to (33.7, 95.2), turned to 180 degrees
- moved C6 103.1 mm to (33.7, 96.8), turned to 180 degrees
- moved SW1 88.5 mm to (44.2, 98.0), turned to 180 degrees
- moved C11 88.4 mm to (31.3, 65.8), turned to 180 degrees
- moved R13 87.5 mm to (27.1, 83.5), turned to 180 degrees
- moved J4 87.4 mm to (27.5, 51.6), turned to -90 degrees
- moved C4 86.7 mm to (38.1, 99.1), turned to -90 degrees
- moved SW2 86.0 mm to (27.9, 78.7), turned to -90 degrees
- moved D2 85.1 mm to (38.7, 34.5), turned to 90 degrees
- moved Q3 83.7 mm to (36.9, 44.9), turned to 90 degrees
- moved D1 79.9 mm to (43.7, 34.5), turned to 90 degrees
- moved R4 79.7 mm to (39.5, 99.0), turned to -90 degrees
- moved C7 79.6 mm to (40.9, 53.8)
- moved U1 79.5 mm to (35.4, 62.4), turned to 180 degrees
- moved U4 76.2 mm to (39.8, 51.4), turned to 180 degrees
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Connections:
- U2 pad 2: RXD1 -> TXD1
- U2 pad 3: TXD1 -> RXD1
- U3 pad 27: unconnected-(U3-IO16-Pad27) -> TXD1
- U3 pad 28: unconnected-(U3-IO17-Pad28) -> RXD1
- U3 pad 30: unconnected-(U3-IO18-Pad30) -> SCK
- U3 pad 31: unconnected-(U3-IO19-Pad31) -> MISO
- U3 pad 36: unconnected-(U3-IO22-Pad36) -> CS_FLASH
- U3 pad 37: unconnected-(U3-IO23-Pad37) -> MOSI
- U3 pad 4: unconnected-(U3-SENSOR_VP-Pad4) -> GPIO_0
Routing:
- net SCK: track 0.00 -> 53.0 mm, vias 0 -> 1
- net MISO: track 0.00 -> 39.6 mm
- net MOSI: track 0.00 -> 37.9 mm, vias 0 -> 1
- net RAW_BATT: track 0.85 -> 29.3 mm
- net CS_FLASH: track 0.00 -> 16.3 mm, vias 0 -> 1
- net RXD1: track 0.00 -> 14.5 mm
- net TXD1: track 0.00 -> 13.0 mm
- net FIRE_A: track 0.00 -> 4.33 mm
- net Net-(Q2-G): track 0.00 -> 2.37 mm
- net Net-(Q3-G): track 0.00 -> 2.04 mm
- net SENSE_A: track 0.00 -> 1.51 mm
- net FIRE_B: track 0.00 -> 1.50 mm
- net SENSE_B: track 0.00 -> 1.50 mm
- net GND: track 0.00 -> 0.62 mm, vias 0 -> 1
- added copper zone on In2.Cu, net +3.3V
- added copper zone on In1.Cu, net GND
- added copper zone on F.Cu, net MOS_A
- added copper zone on F.Cu, net MOS_B
Other:
- board size 31.8 x 88.9 mm -> 31.8 x 76.2 mm
- board text added: "+"
- board text added: "-"

Commit message: V2 finalized
Parts:
- added TP13: TestPoint, TestPoint:TestPoint_Loop_D2.60mm_Drill1.6mm_Beaded, B.Cu at (54.7, 82.3)
- added TP16: TestPoint, TestPoint:TestPoint_Loop_D2.60mm_Drill1.6mm_Beaded, B.Cu at (30.3, 50.6)
- added TP17: TestPoint, TestPoint:TestPoint_Loop_D2.60mm_Drill1.6mm_Beaded, B.Cu at (30.3, 46.3)
- moved TP10 48.3 mm to (43.4, 77.8)
- moved TP11 45.1 mm to (43.4, 72.2)
- moved J3 43.0 mm to (55.2, 92.5)
- moved TP12 42.0 mm to (43.4, 67.9)
- moved TP15 40.6 mm to (43.4, 52.4)
- moved J4 27.4 mm to (54.8, 50.1), turned to 90 degrees
- moved C9 25.6 mm to (55.8, 74.3), turned to -90 degrees
- moved C11 25.2 mm to (54.5, 55.8), turned to 0 degrees
- moved TP4 24.9 mm to (52.7, 86.9)
- moved SW1 23.4 mm to (27.8, 81.3), turned to -90 degrees
- moved U4 23.3 mm to (47.2, 73.5), turned to 90 degrees
- moved R3 21.8 mm to (47.1, 110.5), turned to 0 degrees
- moved C7 21.3 mm to (44.7, 74.8), turned to -90 degrees
- moved SW2 21.2 mm to (27.8, 99.9), turned to 90 degrees
- moved U2 20.8 mm to (31.1, 69.9)
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Connections:
- J4 pad 1: GND -> MISO
- J4 pad 2: +3.3V -> unconnected-(J4-Pin_2-Pad2)
- J4 pad 3: GD00 -> SCK
- J4 pad 4: CS_RF -> MOSI
- J4 pad 5: SCK -> GD00
- J4 pad 6: MOSI -> CS_RF
- J4 pad 7: MISO -> GND
- J4 pad 8: unconnected-(J4-Pin_8-Pad8) -> +3.3V
- U3 pad 10: unconnected-(U3-IO25-Pad10) -> CS_BARO
- U3 pad 11: unconnected-(U3-IO26-Pad11) -> CS_GYRO
- U3 pad 12: unconnected-(U3-IO27-Pad12) -> CS_ACCEL
- U3 pad 13: unconnected-(U3-IO14-Pad13) -> SENSE_A
- U3 pad 14: unconnected-(U3-IO12-Pad14) -> SENSE_B
- U3 pad 16: unconnected-(U3-IO13-Pad16) -> GYRO_INT_A
- U3 pad 23: unconnected-(U3-IO15-Pad23) -> GYRO_INT_B
- U3 pad 24: unconnected-(U3-IO2-Pad24) -> PROGRAM_LED
- U3 pad 25: unconnected-(U3-IO0-Pad25) -> ACCEL_INT_B
- U3 pad 26: unconnected-(U3-IO4-Pad26) -> ACCEL_INT_A
- U3 pad 33: unconnected-(U3-IO21-Pad33) -> MAG_INT
- U3 pad 36: CS_FLASH -> CS_MAG
- U3 pad 6: unconnected-(U3-IO34-Pad6) -> FIRE_A
- U3 pad 7: unconnected-(U3-IO35-Pad7) -> FIRE_B
- U3 pad 8: unconnected-(U3-IO32-Pad8) -> CS_RF
- U3 pad 9: unconnected-(U3-IO33-Pad9) -> CS_FLASH
- U4 pad 1: ACCEL_INT -> ACCEL_INT_B
- U4 pad 12: GYRO_INT -> GYRO_INT_A
- U4 pad 13: GYRO_INT -> GYRO_INT_B
- U4 pad 16: ACCEL_INT -> ACCEL_INT_A
- U5 pad 11: unconnected-(U5-GND-Pad11) -> GND
Routing:
- net SENSE_B: track 1.50 -> 95.4 mm, vias 0 -> 1
- net SENSE_A: track 1.51 -> 80.6 mm, vias 0 -> 1
- net FIRE_A: track 4.33 -> 75.5 mm, vias 0 -> 1
- net FIRE_B: track 1.50 -> 66.0 mm, vias 0 -> 1
- net CS_RF: track 0.00 -> 58.8 mm, vias 0 -> 1
- net MISO: track 39.6 -> 91.1 mm, vias 0 -> 3
- net GYRO_INT_A: track 0.00 -> 49.3 mm, vias 0 -> 4
- net CS_BARO: track 0.00 -> 45.5 mm, vias 0 -> 1
- net ACCEL_INT_B: track 0.00 -> 43.0 mm, vias 0 -> 2
- net CS_ACCEL: track 0.00 -> 42.7 mm, vias 0 -> 2
- net GYRO_INT_B: track 0.00 -> 42.0 mm, vias 0 -> 2
- net CS_GYRO: track 0.00 -> 39.6 mm, vias 0 -> 1
- net GND: track 0.62 -> 40.2 mm, vias 1 -> 28
- net RESET: track 0.00 -> 39.2 mm, vias 0 -> 1
- net ACCEL_INT_A: track 0.00 -> 38.7 mm, vias 0 -> 2
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- added copper zone on F.Cu, net +3.3V
Other:
- board size 31.8 x 76.2 mm -> 31.8 x 88.9 mm
- board text added: "+3.3V"
- board text added: "+5V"
- board text added: "+BATT"
- board text added: "APOGEE"
- board text added: "BATT"
- board text added: "CC1101 RF MODULE"
- board text added: "CS_ACCEL"
- board text added: "CS_BARO"
- board text added: "CS_FLASH"
- board text added: "CS_GYRO"
- board text added: "CS_MAG"
- board text added: "CS_RF"
- board text added: "FIRE_A"
- board text added: "FIRE_B"
- board text added: "GND"
- board text added: "GPIO0"
- board text added: "IN"
- board text added: "MAIN"
- board text added: "MISO"
- board text added: "MOSI"
- board text added: "OUT"
- board text added: "RESET"
- board text added: "RXD0"
- board text added: "RXD1"
- board text added: "SCK"
- board text added: "SENSE_A"
- board text added: "SENSE_B"
- board text added: "SWITCH"
- board text added: "TXD0"
- board text added: "TXD1"
