File: V2/Flight-Computer_V2.kicad_sch (KiCad schematic)
At the start: 62 parts, among them J1 Conn_01x04_Pin, J2 Conn_01x04_Pin, J3 Conn_01x06_Pin, J4 Conn_02x04_Odd_Even, J5 2337019-1, Q1 DMP3099L-7, Q2 NMOS, Q3 NMOS, SW1 PTS636 SM50J SMTR LFS, SW2 PTS636 SM50J SMTR LFS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

Commit message: v2 cahnges
Parts:
- Q2, Q3: footprint SI2302-TP:SOT-23_MCC -> SI2302-TP:SOT-23_MCC-M
Other:
- note added: "needed?"
Changed lines of the file:
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@@
 		)
 	)
+	(text "needed?"
+		(exclude_from_sim no)
+		(at 32.766 198.12 0)
+		(effects
+			(font
+				(size 1.27 1.27)
+			)
+		)
+	)
 	(text "RF Module"
 		(exclude_from_sim no)
@@
 			)
 		)
-		(property "Footprint" "SI2302-TP:SOT-23_MCC"
+		(property "Footprint" "SI2302-TP:SOT-23_MCC-M"
 			(at 331.47 222.25 0)
 			(effects
@@
 			)
 		)
-		(property "Footprint" "SI2302-TP:SOT-23_MCC"
+		(property "Footprint" "SI2302-TP:SOT-23_MCC-M"
 			(at 331.47 182.88 0)
 			(effects

Commit message: V2 Changes
Parts:
- D1, D2, D3: footprint LED_SMD:LED_0201_0603Metric -> LED_SMD:LED_0402_1005Metric
- TP10, TP11, TP12, TP14, TP15, TP3, TP4, TP5, TP6, TP7, TP8, TP9: footprint TestPoint:TestPoint_Loop_D1.80mm_Drill1.0mm_Beaded -> TestPoint:TestPoint_Loop_D2.60mm_Drill1.6mm_Beaded
Connections:
- net CS_FLASH: now also U3.36 (IO22)
- net GPIO_0: now also U3.4 (SENSOR_VP)
- net MISO: now also U3.31 (IO19)
- net MOSI: now also U3.37 (IO23)
- net RXD1: now also U2.3 (RXD), U3.28 (IO17); no longer U2.2 (TXD)
- net SCK: now also U3.30 (IO18)
- net TXD1: now also U2.2 (TXD), U3.27 (IO16); no longer U2.3 (RXD)
Other:
- note added: "make smaller"
Changed lines of the file:
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@@
 		)
 	)
+	(text "make smaller"
+		(exclude_from_sim no)
+		(at 69.596 259.08 0)
+		(effects
+			(font
+				(size 1.27 1.27)
+			)
+		)
+	)
 	(text "needed?"
 		(exclude_from_sim no)
@@
 	(wire
 		(pts
+			(xy 193.04 140.97) (xy 196.85 140.97)
+		)
+		(stroke
+			(width 0)
+			(type default)
+		)
+	)
+	(wire
+		(pts
 			(xy 360.68 100.33) (xy 364.49 100.33)
 		)
@@
 	(wire
 		(pts
+			(xy 227.33 163.83) (xy 231.14 163.83)
+		)
+		(stroke
+			(width 0)
+			(type default)
+		)
+	)
+	(wire
+		(pts
 			(xy 64.77 165.1) (xy 64.77 162.56)
 		)
@@
 	(wire
 		(pts
+			(xy 227.33 176.53) (xy 231.14 176.53)
+		)
+		(stroke
+			(width 0)
+			(type default)
+		)
+	)
+	(wire
+		(pts
 			(xy 311.15 48.26) (xy 308.61 48.26)
 		)
@@
 	(wire
 		(pts
+			(xy 227.33 161.29) (xy 231.14 161.29)
+		)
+		(stroke
+			(width 0)
+			(type default)
+		)
+	)
+	(wire
+		(pts
 			(xy 292.1 55.88) (xy 292.1 59.69)
 		)
@@
 	(wire
 		(pts
+			(xy 227.33 168.91) (xy 231.14 168.91)
+		)
+		(stroke
+			(width 0)
+			(type default)
+		)
+	)
+	(wire
+		(pts
 			(xy 339.09 217.17) (xy 339.09 205.74)
 		)
@@
 	(wire
 		(pts
+			(xy 227.33 166.37) (xy 231.14 166.37)
+		)
+		(stroke
+			(width 0)
+			(type default)
+		)
+	)
+	(wire
+		(pts
 			(xy 339.09 232.41) (xy 351.79 232.41)
 		)
@@
 	(wire
 		(pts
+			(xy 227.33 173.99) (xy 231.14 173.99)
+		)
+		(stroke
+			(width 0)
+			(type default)
+		)
+	)
+	(wire
+		(pts
 			(xy 361.95 48.26) (xy 381 48.26)
 		)
@@
 		)
 	)
+	(global_label "SCK"
+		(shape input)
+		(at 231.14 166.37 0)
+		(fields_autoplaced yes)
+		(effects
+			(font
+				(size 1.27 1.27)
+			)
+			(justify left)
+		)
+		(property "Intersheetrefs" "${INTERSHEET_REFS}"
+			(at 237.8747 166.37 0)
+			(effects
+				(font
+					(size 1.27 1.27)
+				)
+				(justify left)
+				(hide yes)
+			)
+		)
+	)
 	(global_label "FIRE_B"
 		(shape input)
@@
 		)
 	)
+	(global_label "RXD1"
+		(shape input)
+		(at 231.14 163.83 0)
+		(fields_autoplaced yes)
+		(effects
+			(font
+				(size 1.27 1.27)
+			)
+			(justify left)
+		)
+		(property "Intersheetrefs" "${INTERSHEET_REFS}"
+			(at 239.0842 163.83 0)
+			(effects
+				(font
+					(size 1.27 1.27)
+				)
+				(justify left)
+				(hide yes)
+			)
+		)
+	)
 	(global_label "MOS_A"
 		(shape input)
@@
 	(global_label "RXD1"
 		(shape input)
-		(at 186.69 53.34 180)
+		(at 186.69 50.8 180)
 		(fields_autoplaced yes)
 		(effects
@@
 		)
 		(property "Intersheetrefs" "${INTERSHEET_REFS}"
-			(at 178.7458 53.34 0)
+			(at 178.7458 50.8 0)
 			(effects
 				(font
@@
 		)
 	)
+	(global_label "TXD1"
+		(shape input)
+		(at 231.14 161.29 0)
+		(fields_autoplaced yes)
+		(effects
+			(font
+				(size 1.27 1.27)
+			)
+			(justify left)
+		)
+		(property "Intersheetrefs" "${INTERSHEET_REFS}"
+			(at 238.7818 161.29 0)
+			(effects
+				(font
+					(size 1.27 1.27)
+				)
+				(justify left)
+				(hide yes)
+			)
+		)
+	)
 	(global_label "CS_RF"
 		(shape input)
@@
 	(global_label "MISO"
 		(shape input)
+		(at 231.14 168.91 0)
+		(fields_autoplaced yes)
+		(effects
+			(font
+				(size 1.27 1.27)
+			)
+			(justify left)
+		)
+		(property "Intersheetrefs" "${INTERSHEET_REFS}"
+			(at 238.7214 168.91 0)
+			(effects
+				(font
+					(size 1.27 1.27)
+				)
+				(justify left)
+				(hide yes)
+			)
+		)
+	)
+	(global_label "MISO"
+		(shape input)
 		(at 308.61 95.25 180)
 		(fields_autoplaced yes)
@@
 		)
 	)
+	(global_label "MOSI"
+		(shape input)
+		(at 231.14 176.53 0)
+		(fields_autoplaced yes)
+		(effects
+			(font
+				(size 1.27 1.27)
+			)
+			(justify left)
+		)
+		(property "Intersheetrefs" "${INTERSHEET_REFS}"
+			(at 238.7214 176.53 0)
+			(effects
+				(font
+					(size 1.27 1.27)
+				)
+				(justify left)
+				(hide yes)
+			)
+		)
+	)
 	(global_label "GYRO_INT"
 		(shape input)
@@
 	(global_label "CS_FLASH"
 		(shape input)
-		(at 171.45 158.75 180)
+		(at 231.14 173.99 0)
 		(fields_autoplaced yes)
 		(effects
@@
 				(size 1.27 1.27)
 			)
-			(justify right)
+			(justify left)
 		)
 		(property "Intersheetrefs" "${INTERSHEET_REFS}"
-			(at 159.2724 158.75 0)
+			(at 243.3176 173.99 0)
 			(effects
 				(font
 					(size 1.27 1.27)
 				)
-				(justify right)
+				(justify left)
 				(hide yes)
 			)
@@
 	(global_label "TXD1"
 		(shape input)
-		(at 186.69 50.8 180)
+		(at 186.69 53.34 180)
 		(fields_autoplaced yes)
 		(effects
@@
 		)
 		(property "Intersheetrefs" "${INTERSHEET_REFS}"
-			(at 179.0482 50.8 0)
+			(at 179.0482 53.34 0)
 			(effects
 				(font
@@
 			)
 		)
-		(property "Footprint" "TestPoint:TestPoint_Loop_D1.80mm_Drill1.0mm_Beaded"
+		(property "Footprint" "TestPoint:TestPoint_Loop_D2.60mm_Drill1.6mm_Beaded"
 			(at 31.75 241.3 0)
 			(effects
@@
 			)
 		)
-		(property "Footprint" "TestPoint:TestPoint_Loop_D1.80mm_Drill1.0mm_Beaded"
+		(property "Footprint" "TestPoint:TestPoint_Loop_D2.60mm_Drill1.6mm_Beaded"
 			(at 46.99 264.16 0)
 			(effects
@@
 			)
 		)
-		(property "Footprint" "TestPoint:TestPoint_Loop_D1.80mm_Drill1.0mm_Beaded"
+		(property "Footprint" "TestPoint:TestPoint_Loop_D2.60mm_Drill1.6mm_Beaded"
 			(at 24.13 264.16 0)
 			(effects
@@
 			)
 		)
-		(property "Footprint" "TestPoint:TestPoint_Loop_D1.80mm_Drill1.0mm_Beaded"
+		(property "Footprint" "TestPoint:TestPoint_Loop_D2.60mm_Drill1.6mm_Beaded"
 			(at 39.37 241.3 0)
 			(effects
@@
 			)
 		)
-		(property "Footprint" "LED_SMD:LED_0201_0603Metric"
+		(property "Footprint" "LED_SMD:LED_0402_1005Metric"
 			(at 111.76 49.53 0)
 			(effects
@@
 			)
 		)
-		(property "Footprint" "TestPoint:TestPoint_Loop_D1.80mm_Drill1.0mm_Beaded"
+		(property "Footprint" "TestPoint:TestPoint_Loop_D2.60mm_Drill1.6mm_Beaded"
 			(at 46.99 241.3 0)
 			(effects
@@
 			)
 		)
-		(property "Footprint" "TestPoint:TestPoint_Loop_D1.80mm_Drill1.0mm_Beaded"
+		(property "Footprint" "TestPoint:TestPoint_Loop_D2.60mm_Drill1.6mm_Beaded"
 			(at 54.61 264.16 0)
 			(effects
@@
 			)
 		)
-		(property "Footprint" "TestPoint:TestPoint_Loop_D1.80mm_Drill1.0mm_Beaded"
+		(property "Footprint" "TestPoint:TestPoint_Loop_D2.60mm_Drill1.6mm_Beaded"
 			(at 69.85 241.3 0)
 			(effects
@@
 			)
 		)
-		(property "Footprint" "TestPoint:TestPoint_Loop_D1.80mm_Drill1.0mm_Beaded"
+		(property "Footprint" "TestPoint:TestPoint_Loop_D2.60mm_Drill1.6mm_Beaded"
 			(at 54.61 241.3 0)
 			(effects
@@
 			)
 		)
-		(property "Footprint" "TestPoint:TestPoint_Loop_D1.80mm_Drill1.0mm_Beaded"
+		(property "Footprint" "TestPoint:TestPoint_Loop_D2.60mm_Drill1.6mm_Beaded"
 			(at 16.51 264.16 0)
 			(effects
@@
 			)
 		)
-		(property "Footprint" "TestPoint:TestPoint_Loop_D1.80mm_Drill1.0mm_Beaded"
+		(property "Footprint" "TestPoint:TestPoint_Loop_D2.60mm_Drill1.6mm_Beaded"
 			(at 31.75 264.16 0)
 			(effects
@@
 			)
 		)
-		(property "Footprint" "TestPoint:TestPoint_Loop_D1.80mm_Drill1.0mm_Beaded"
+		(property "Footprint" "TestPoint:TestPoint_Loop_D2.60mm_Drill1.6mm_Beaded"
 			(at 77.47 241.3 0)
 			(effects
@@
 			)
 		)
-		(property "Footprint" "LED_SMD:LED_0201_0603Metric"
+		(property "Footprint" "LED_SMD:LED_0402_1005Metric"
 			(at 135.89 49.53 0)
 			(effects
@@
 			)
 		)
-		(property "Footprint" "LED_SMD:LED_0201_0603Metric"
+		(property "Footprint" "LED_SMD:LED_0402_1005Metric"
 			(at 123.19 49.53 0)
 			(effects
@@
 			)
 		)
-		(property "Footprint" "TestPoint:TestPoint_Loop_D1.80mm_Drill1.0mm_Beaded"
+		(property "Footprint" "TestPoint:TestPoint_Loop_D2.60mm_Drill1.6mm_Beaded"
 			(at 62.23 241.3 0)
 			(effects

Commit message: V2 finalized
Parts:
- added TP13, TP16, TP17: TestPoint, TestPoint:TestPoint_Loop_D2.60mm_Drill1.6mm_Beaded, symbol Connector:TestPoint
Connections:
- net +3.3V: now also J4.8 (Pin_8); no longer J4.2 (Pin_2)
- net ACCEL_INT: no longer U4.1 (INT2), U4.16 (INT1)
- net CS_ACCEL: now also U3.12 (IO27)
- net CS_BARO: now also U3.10 (IO25)
- net CS_FLASH: now also U3.9 (IO33); no longer U3.36 (IO22)
- net CS_GYRO: now also U3.11 (IO26)
- net CS_MAG: now also U3.36 (IO22), TP13.1
- net CS_RF: now also J4.6 (Pin_6), U3.8 (IO32); no longer J4.4 (Pin_4)
- net FIRE_A: now also U3.6 (IO34)
- net FIRE_B: now also U3.7 (IO35)
- net GD00: now also J4.5 (Pin_5); no longer J4.3 (Pin_3)
- net GND: now also J4.7 (Pin_7), U5.11 (GND); no longer J4.1 (Pin_1)
- net MAG_INT: now also U3.33 (IO21)
- net MISO: now also J4.1 (Pin_1); no longer J4.7 (Pin_7)
- net MOSI: now also J4.4 (Pin_4); no longer J4.6 (Pin_6)
- net PROGRAM_LED: now also U3.24 (IO2)
- net SCK: now also J4.3 (Pin_3); no longer J4.5 (Pin_5)
- net SENSE_A: now also U3.13 (IO14), TP16.1
- net SENSE_B: now also U3.14 (IO12), TP17.1
- net GYRO_INT_A: now reaches U3.16 (IO13)
- net GYRO_INT_A: now also U4.12 (INT3)
- net GYRO_INT_B: now reaches U3.23 (IO15)
- net GYRO_INT_B: now also U4.13 (INT4)
- net ACCEL_INT_B: now reaches U3.25 (IO0)
- net ACCEL_INT_B: now also U4.1 (INT2)
- net ACCEL_INT_A: now reaches U3.26 (IO4)
- net ACCEL_INT_A: now also U4.16 (INT1)
- removed net GYRO_INT: U4.12 (INT3), U4.13 (INT4)
Other:
- note removed: "make smaller"
