File: V3/V3/V3.kicad_pcb (KiCad board)
At the start: 2 copper layers, 31.8 x 38.1 mm, 65 parts, among them J1 Conn_01x04_Pin, J2 Conn_01x04_Pin, J3 Conn_01x06_Pin, J4 Conn_01x07_Pin, J5 2337019-1, Q1 DMP3099L-7, Q2 NMOS, Q3 NMOS, SW1 PTS636 SM50J SMTR LFS, SW2 PTS636 SM50J SMTR LFS, U1 W25Q16JVSSIQ, U2 MAX-M10M-00B, U3 ESP32-WROOM-32UE, U4 BMI088, U5 MMC5983MA, U6 MS560702BA03-50

Commit message: V3 changes
Parts:
- removed TP15: TestPoint, RCU_0C:CONN1_RCU-0C_TEC
- BMI088 : renamed from U4
- moved TP14 22.7 mm to (40.2, 42.5), turned to 90 degrees
- moved TP11 19.5 mm to (42.2, 49.0), turned to 90 degrees
- moved J5 18.9 mm to (40.9, 55.6), turned to -90 degrees
- moved TP13 17.9 mm to (49.3, 41.2), turned to 180 degrees
- moved J4 15.2 mm to (33.7, 61.7), turned to 90 degrees
- moved J3 12.9 mm to (55.3, 46.2), turned to 0 degrees
- moved TP10 12.7 mm to (47.5, 52.2), turned to 180 degrees
- moved TP12 12.1 mm to (55.9, 48.8), turned to 0 degrees
- moved R14 2.30 mm to (41.4, 43.7), turned to -90 degrees
- moved R3 2.28 mm to (51.4, 34.8), turned to 90 degrees
- moved LDO 1.51 mm to (40.0, 27.7), turned to 90 degrees
- moved C6 1.34 mm to (35.6, 57.7), turned to -90 degrees
- moved C1 1.22 mm to (37.5, 28.2)
- moved TP17 1.22 mm to (29.1, 37.3)
- moved C8 1.00 mm to (47.7, 36.8)
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- renumbered TP1 to +3V3, TP2 to +BATT, U6 to BARO, U1 to FLASH, U2 to GPS, CR1 to LDO, U5 to MAG
Connections:
- U3 pad 16: GYRO_INT_A -> CS_FLASH
- U3 pad 23: RF_INT -> MAG_INT
- U3 pad 25: ACCEL_INT_B -> CS_BARO
- U3 pad 26: CS_FLASH -> CS_GYRO
- U3 pad 29: CS_GYRO -> GYRO_INT_A
- U3 pad 33: MAG_INT -> CS_ACCEL
- U3 pad 36: CS_ACCEL -> ACCEL_INT_A
- U3 pad 5: CS_MAG -> RF_INT
- U3 pad 6: ACCEL_INT_A -> GYRO_INT_B
- U3 pad 7: CS_BARO -> ACCEL_INT_B
- U3 pad 8: GYRO_INT_B -> CS_MAG
Routing:
- net RESET: track 7.73 -> 48.8 mm
- net GPIO_0: track 11.2 -> 49.9 mm, vias 0 -> 3
- net GND: track 0.00 -> 34.4 mm, vias 0 -> 29
- net RAW_BATT: track 0.00 -> 29.5 mm
- net CS_MAG: track 0.00 -> 26.1 mm, vias 0 -> 1
- net RF_INT: track 0.00 -> 23.8 mm, vias 0 -> 1
- net TXD2: track 0.00 -> 22.6 mm, vias 0 -> 1
- net CS_BARO: track 0.00 -> 22.3 mm, vias 0 -> 1
- net +3.3V: track 0.00 -> 22.2 mm, vias 0 -> 15
- net RXD2: track 0.00 -> 20.2 mm, vias 0 -> 1
- net TXD0: track 0.00 -> 14.5 mm, vias 0 -> 1
- net GYRO_INT_B: track 0.64 -> 15.0 mm, vias 0 -> 1
- net CS_GYRO: track 0.00 -> 13.3 mm, vias 0 -> 3
- net RXD0: track 0.00 -> 13.2 mm, vias 0 -> 1
- net ACCEL_INT_B: track 0.00 -> 12.3 mm, vias 0 -> 1
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- added copper zone on In2.Cu, net +3.3V
- added copper zone on B.Cu, net +BATT
- added copper zone on In1.Cu, net GND
Other:
- copper layers 2 -> 4
- board text added: "+5V"
- board text added: "- +"
- board text added: "CS FLSH"
- board text added: "CS_ACCEL"
- board text added: "FIRE_A"
- board text added: "FIRE_B"
- board text added: "GND"
- board text added: "GPIO0"
- board text added: "LiPO"
- board text added: "MISO"
- board text added: "MOSI"
- board text added: "RF ANT"
- board text added: "RST"
- board text added: "RXD0"
- board text added: "RXD1"
- board text added: "SCK"
- board text added: "SENSE_B"
- board text added: "TXD0"
- board text added: "TXD1"
